File: WeMos-Matrix-Shield.brd (EAGLE design)
At the start: 36.2 x 47 mm, 13 parts, among them CN1 1X4-BIG, J2 POWER_JACKPTH, X1 SPTAF_23.5

Commit message: Bump to V1.1
Parts:
- removed JP5, JP9: (no value), SparkFun-Connectors:1X02_NO_SILK
- removed U$2: (no value), _c2h:LOGO_C2I_015
- added J3: (no value), SparkFun-Connectors:SCREWTERMINAL-3.5MM-4
- added U$3: (no value), _c2h:LOGO_CH2I_110MM
- U$1: device _c2h:LOGO_C2I_015 -> _c2h:LOGO_CH2I_110MM
- X1: value SPTAF_23.5 -> SPTAF_25.0MM; device _c2h:FFKV2_35 -> _c2h:SPTAF_2X50
- moved J1 36.2 mm to (50.2, 47.4)
- moved U$1 21.3 mm to (48.3, 9.53), flipped to the bottom
- moved CN1 1.27 mm to (40.6, 7.62)
- moved X1 0.63 mm to (32.4, 12.1)
Connections:
- net 5V: now also J3.1, J3.2; no longer JP9.1, JP9.2
- net B0: now also J1.6; no longer J1.3
- net B1: now also J1.3
- net G0: now also J1.5; no longer J1.2
- net G1: now also J1.2; no longer J1.6
- net GND: now also J3.3, J3.4; no longer JP5.1, JP5.2
- net R0: no longer J1.1
- net R1: now also J1.1; no longer J1.5
Routing:
- net B1: track 0.00 -> 53.9 mm
- net B0: track 16.1 -> 60.7 mm
- net R1: track 14.8 -> 57.1 mm
- net G1: track 14.8 -> 53.3 mm, vias 0 -> 1
- net 5V: track 93.4 -> 62.3 mm
- net G0: track 16.1 -> 43.9 mm
- net R0: track 25.1 -> 12.2 mm
- net E: track 37.0 -> 38.2 mm
- net C: track 25.1 -> 26.0 mm
- net STB: track 38.1 -> 37.5 mm
- net GND: vias 6 -> 20
Other:
- board size 36.2 x 47 mm -> 45.1 x 47 mm
- board text added: "Output"
- board text added: "R0 -- D7/GPIO13 E --- D7/GPIO0 A --- D1/GPIO5 B --- D2/GPIO4 C --- D8/GPIO15 D --- D6/GPIO12 CLK - D5/GPIO14 STB - D0/GPIO16 OE -- D4/GPIO2"
- board text added: "WeMos Matrix Shield V1.1"
- board text added: "github.com/hallard"
- board text removed: "To Out"
- board text removed: "WeMos Matrix Shield V1.0"

Commit message: Update to V1.2
Parts:
- added C1: 100nF, _c2h:CAP-PTH-SMALL2
- added R1: 10K, _c2h:1/6W-RES
- added U1: LDR, Seeed-Sensor:SNR2-3.0
Connections:
- net 3V3: now also U1.2
- net A0: now also C1.1, R1.2, U1.1
- net GND: now also C1.2, R1.1
Routing:
- net 3V3: track 2.54 -> 38.0 mm, vias 0 -> 1
- net A0: track 2.54 -> 35.5 mm
- net G1: track 53.3 -> 39.3 mm
- net G0: track 43.9 -> 42.8 mm
- net GND: vias 20 -> 21
Other:
- board text added: "WeMos Matrix Shield V1.2"
- board text removed: "WeMos Matrix Shield V1.1"
Changed lines of the file:
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@@
 Matrix
 Shield
-V1.1</text>
+V1.2</text>
 <text x="11.714" y="36.20025" size="0.889" layer="25" font="vector" ratio="15" rot="R180" align="center">R0</text>
 <text x="11.714" y="26.04025" size="0.889" layer="25" font="vector" ratio="15" rot="R180" align="center">A</text>
@@
 <text x="25.01375" y="15.27" size="0.889" layer="26" font="vector" ratio="15" rot="MR270" align="center">5V</text>
 <text x="33.05175" y="47.244" size="1.397" layer="26" font="vector" ratio="15" rot="MR0" align="center">WeMos Matrix Shield
-V1.1</text>
+V1.2</text>
 <text x="29.815" y="16.12375" size="0.889" layer="26" font="vector" ratio="15" rot="MR180" align="center">GND</text>
 <text x="35.022" y="16.12375" size="0.889" layer="26" font="vector" ratio="15" rot="MR180" align="center">5V</text>
@@
 <wire x1="53.34" y1="49.911" x2="53.34" y2="49.657" width="0.3048" layer="25"/>
 <wire x1="51.308" y1="49.911" x2="52.832" y2="49.911" width="0.4064" layer="25"/>
-<text x="50.79825" y="50.42425" size="0.889" layer="25" font="vector" ratio="15" rot="R180">Output</text>
-<text x="15.23825" y="40.01025" size="0.889" layer="25" font="vector" ratio="15" rot="R180" align="center">Input</text>
+<text x="51.05225" y="50.55125" size="1.016" layer="25" font="vector" ratio="15" rot="R180">Output</text>
+<text x="13.20625" y="39.62925" size="1.016" layer="25" font="vector" ratio="15" rot="R180" align="center">Input</text>
 <text x="40.03675" y="34.798" size="1.016" layer="26" ratio="15" rot="MR0" align="center-left">R0 -- D7/GPIO13
 E --- D7/GPIO0
@@
 <element name="U$3" library="_c2h" package="LOGO_CH2I_110MM" value="" x="49.53" y="9.525"/>
 <element name="U$1" library="_c2h" package="LOGO_CH2I_110MM" value="" x="48.26" y="9.525" rot="MR0"/>
+<element name="U1" library="Seeed-Sensor" package="SNR2-3.0" value="LDR" x="52.07" y="36.83" smashed="yes" rot="R270">
+<attribute name="MPN" value="PHOTORESISTOR-5528-10K" x="52.07" y="36.83" size="1.778" layer="27" font="vector" ratio="15" rot="R270" display="off"/>
+<attribute name="VALUE" x="50.546" y="36.83" size="0.8128" layer="25" font="vector" ratio="15" rot="R90" align="center"/>
+</element>
+<element name="R1" library="_c2h" package="1/6W-RES" value="10K" x="48.26" y="36.83" smashed="yes" rot="R90">
+<attribute name="NAME" x="46.228" y="37.592" size="0.8128" layer="25" font="vector" ratio="15" rot="R270"/>
+<attribute name="VALUE" x="48.641" y="35.814" size="0.8128" layer="21" font="vector" ratio="15" rot="R90"/>
+</element>
+<element name="C1" library="_c2h" package="CAP-PTH-SMALL2" value="100nF" x="19.05" y="41.91" smashed="yes" rot="R270">
+<attribute name="NAME" x="17.018" y="40.767" size="0.8128" layer="25" font="vector" ratio="15" rot="R90" align="center"/>
+</element>
 </elements>
 <signals>
@@
 <via x="34.925" y="41.91" extent="1-16" drill="0.3556" diameter="0.7112"/>
 <via x="12.7" y="40.64" extent="1-16" drill="0.3556" diameter="0.7112"/>
-<via x="45.085" y="16.51" extent="1-16" drill="0.3556" diameter="0.7112"/>
+<via x="43.18" y="6.985" extent="1-16" drill="0.3556" diameter="0.7112"/>
 <via x="39.37" y="49.784" extent="1-16" drill="0.3556" diameter="0.7112"/>
 <via x="24.638" y="49.911" extent="1-16" drill="0.3556" diameter="0.7112"/>
@@
 <contactref element="J3" pad="4"/>
 <via x="40.64" y="23.495" extent="1-16" drill="0.3556" diameter="0.7112"/>
-<via x="50.165" y="37.465" extent="1-16" drill="0.3556" diameter="0.7112"/>
-<via x="31.75" y="27.305" extent="1-16" drill="0.3556" diameter="0.7112"/>
+<via x="46.99" y="41.275" extent="1-16" drill="0.3556" diameter="0.7112"/>
+<via x="31.115" y="27.94" extent="1-16" drill="0.3556" diameter="0.7112"/>
 <via x="30.48" y="44.45" extent="1-16" drill="0.3556" diameter="0.7112"/>
 <via x="18.669" y="49.149" extent="1-16" drill="0.3556" diameter="0.7112"/>
@@
 <via x="27.051" y="30.099" extent="1-16" drill="0.3556" diameter="0.7112"/>
 <via x="27.051" y="36.576" extent="1-16" drill="0.3556" diameter="0.7112"/>
-<via x="16.764" y="40.767" extent="1-16" drill="0.3556" diameter="0.7112"/>
+<via x="15.494" y="40.767" extent="1-16" drill="0.3556" diameter="0.7112"/>
 <via x="22.86" y="25.146" extent="1-16" drill="0.3556" diameter="0.7112"/>
 <via x="19.685" y="28.956" extent="1-16" drill="0.3556" diameter="0.7112"/>
 <via x="19.05" y="22.225" extent="1-16" drill="0.3556" diameter="0.7112"/>
 <via x="21.59" y="21.082" extent="1-16" drill="0.3556" diameter="0.7112"/>
-<via x="19.177" y="43.053" extent="1-16" drill="0.3556" diameter="0.7112"/>
+<via x="14.732" y="44.323" extent="1-16" drill="0.3556" diameter="0.7112"/>
+<contactref element="R1" pad="1"/>
+<via x="31.115" y="25.4" extent="1-16" drill="0.3556" diameter="0.7112"/>
+<contactref element="C1" pad="2"/>
 </signal>
 <signal name="3V3">
@@
 <contactref element="JP7" pad="8"/>
 <wire x1="24.13" y1="26.67" x2="21.59" y2="26.67" width="0.6096" layer="16"/>
+<contactref element="U1" pad="2"/>
+<wire x1="52.07" y1="35.179" x2="51.181" y2="35.179" width="0.3048" layer="16"/>
+<wire x1="51.181" y1="35.179" x2="50.8" y2="35.56" width="0.3048" layer="16"/>
+<wire x1="50.8" y1="35.56" x2="36.195" y2="35.56" width="0.3048" layer="16"/>
+<wire x1="36.195" y1="35.56" x2="35.56" y2="34.925" width="0.3048" layer="16"/>
+<via x="35.56" y="34.925" extent="1-16" drill="0.3556" diameter="0.7112"/>
+<wire x1="35.56" y1="34.925" x2="35.56" y2="28.575" width="0.3048" layer="1"/>
+<wire x1="35.56" y1="28.575" x2="33.655" y2="26.67" width="0.3048" layer="1"/>
+<wire x1="33.655" y1="26.67" x2="24.13" y2="26.67" width="0.3048" layer="1"/>
 </signal>
 <signal name="A0">
@@
 <contactref element="JP7" pad="2"/>
 <wire x1="24.13" y1="41.91" x2="21.59" y2="41.91" width="0.6096" layer="16"/>
+<contactref element="U1" pad="1"/>
+<contactref element="R1" pad="2"/>
+<wire x1="47.03" y1="38.1" x2="30.48" y2="38.1" width="0.3048" layer="16"/>
+<wire x1="30.48" y1="38.1" x2="26.67" y2="41.91" width="0.3048" layer="16"/>
+<wire x1="26.67" y1="41.91" x2="24.13" y2="41.91" width="0.3048" layer="16"/>
+<wire x1="47.03" y1="38.1" x2="48.26" y2="39.33" width="0.3048" layer="16"/>
+<wire x1="48.26" y1="39.33" x2="51.221" y2="39.33" width="0.3048" layer="16"/>
+<wire x1="51.221" y1="39.33" x2="52.07" y2="38.481" width="0.3048" layer="16"/>
+<contactref element="C1" pad="1"/>
+<wire x1="19.05" y1="41.91" x2="21.59" y2="41.91" width="0.3048" layer="16"/>
 </signal>
 <signal name="STB">
@@
 <signal name="G0">
 <contactref element="JP2" pad="2"/>
-<wire x1="19.939" y1="37.719" x2="18.415" y2="36.195" width="0.3048" layer="16"/>
-<wire x1="18.415" y1="36.195" x2="16.51" y2="36.195" width="0.3048" layer="16"/>
-<wire x1="19.939" y1="37.719" x2="19.939" y2="45.339" width="0.3048" layer="16"/>
 <contactref element="J1" pad="5"/>
-<wire x1="19.939" y1="45.339" x2="20.828" y2="46.228" width="0.3048" layer="16"/>
 <wire x1="20.828" y1="46.228" x2="45.212" y2="46.228" width="0.3048" layer="16"/>
 <wire x1="45.212" y1="46.228" x2="49.149" y2="42.291" width="0.3048" layer="16"/>
 <wire x1="50.165" y1="42.291" x2="49.149" y2="42.291" width="0.3048" layer="16"/>
+<wire x1="20.828" y1="46.228" x2="16.51" y2="41.91" width="0.3048" layer="16"/>
+<wire x1="16.51" y1="41.91" x2="16.51" y2="36.195" width="0.3048" layer="16"/>
 </signal>
 <signal name="G1">
@@
 <wire x1="17.78" y1="31.115" x2="16.51" y2="31.115" width="0.3048" layer="1"/>
 <contactref element="J1" pad="2"/>
-<wire x1="18.415" y1="31.75" x2="18.415" y2="45.72" width="0.3048" layer="1"/>
 <via x="18.415" y="45.72" extent="1-16" drill="0.3556" diameter="0.7112"/>
 <wire x1="18.415" y1="45.72" x2="18.415" y2="46.355" width="0.3048" layer="16"/>
@@
 <wire x1="52.07" y1="48.895" x2="52.705" y2="48.26" width="0.3048" layer="16"/>
 <wire x1="52.705" y1="48.26" x2="52.705" y2="47.371" width="0.3048" layer="16"/>
+<wire x1="18.415" y1="31.75" x2="18.415" y2="45.72" width="0" layer="19" extent="1-1"/>
 </signal>
 <signal name="E">

Commit message: Updated to V1.3
Routing:
- net G1: track 39.3 -> 54.0 mm
- net R0: track 12.2 -> 13.1 mm
- net 3V3: track 38.0 -> 38.8 mm
- net GND: vias 21 -> 22
Other:
- board text added: "WeMos Matrix Shield V1.3"
- board text removed: "WeMos Matrix Shield V1.2"
Changed lines of the file:
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@@
 Matrix
 Shield
-V1.2</text>
+V1.3</text>
 <text x="11.714" y="36.20025" size="0.889" layer="25" font="vector" ratio="15" rot="R180" align="center">R0</text>
 <text x="11.714" y="26.04025" size="0.889" layer="25" font="vector" ratio="15" rot="R180" align="center">A</text>
@@
 <text x="25.01375" y="15.27" size="0.889" layer="26" font="vector" ratio="15" rot="MR270" align="center">5V</text>
 <text x="33.05175" y="47.244" size="1.397" layer="26" font="vector" ratio="15" rot="MR0" align="center">WeMos Matrix Shield
-V1.2</text>
+V1.3</text>
 <text x="29.815" y="16.12375" size="0.889" layer="26" font="vector" ratio="15" rot="MR180" align="center">GND</text>
 <text x="35.022" y="16.12375" size="0.889" layer="26" font="vector" ratio="15" rot="MR180" align="center">5V</text>
@@
 <via x="31.115" y="25.4" extent="1-16" drill="0.3556" diameter="0.7112"/>
 <contactref element="C1" pad="2"/>
+<via x="19.05" y="31.877" extent="1-16" drill="0.3556" diameter="0.7112"/>
 </signal>
 <signal name="3V3">
@@
 <wire x1="36.195" y1="35.56" x2="35.56" y2="34.925" width="0.3048" layer="16"/>
 <via x="35.56" y="34.925" extent="1-16" drill="0.3556" diameter="0.7112"/>
-<wire x1="35.56" y1="34.925" x2="35.56" y2="28.575" width="0.3048" layer="1"/>
-<wire x1="35.56" y1="28.575" x2="33.655" y2="26.67" width="0.3048" layer="1"/>
-<wire x1="33.655" y1="26.67" x2="24.13" y2="26.67" width="0.3048" layer="1"/>
+<wire x1="35.56" y1="34.925" x2="35.56" y2="27.305" width="0.3048" layer="1"/>
+<wire x1="35.56" y1="27.305" x2="34.925" y2="26.67" width="0.3048" layer="1"/>
+<wire x1="34.925" y1="26.67" x2="24.13" y2="26.67" width="0.3048" layer="1"/>
 </signal>
 <signal name="A0">
@@
 <wire x1="15.24" y1="34.925" x2="19.05" y2="34.925" width="0.3048" layer="16"/>
 <wire x1="19.05" y1="34.925" x2="19.685" y2="34.29" width="0.3048" layer="16"/>
-<wire x1="19.685" y1="34.29" x2="21.59" y2="31.75" width="0.3048" layer="16"/>
+<wire x1="21.59" y1="31.75" x2="20.32" y2="31.75" width="0.3048" layer="16"/>
+<wire x1="20.32" y1="31.75" x2="19.685" y2="32.385" width="0.3048" layer="16"/>
+<wire x1="19.685" y1="32.385" x2="19.685" y2="34.29" width="0.3048" layer="16"/>
 </signal>
 <signal name="B0">
@@
 <contactref element="JP7" pad="4"/>
 <wire x1="24.13" y1="36.83" x2="21.59" y2="36.83" width="0.6096" layer="16"/>
-<wire x1="19.685" y1="31.115" x2="19.685" y2="36.195" width="0.3048" layer="1"/>
-<wire x1="19.685" y1="36.195" x2="20.32" y2="36.83" width="0.3048" layer="1"/>
+<wire x1="19.812" y1="31.115" x2="19.812" y2="36.322" width="0.3048" layer="1"/>
+<wire x1="19.812" y1="36.322" x2="20.32" y2="36.83" width="0.3048" layer="1"/>
 <wire x1="20.32" y1="36.83" x2="21.59" y2="36.83" width="0.3048" layer="1"/>
 <wire x1="13.97" y1="20.955" x2="12.7" y2="20.955" width="0.3048" layer="1"/>
@@
 <wire x1="12.065" y1="29.21" x2="12.7" y2="29.845" width="0.3048" layer="1"/>
 <wire x1="12.7" y1="29.845" x2="18.415" y2="29.845" width="0.3048" layer="1"/>
-<wire x1="18.415" y1="29.845" x2="19.685" y2="31.115" width="0.3048" layer="1"/>
+<wire x1="18.415" y1="29.845" x2="19.812" y2="31.115" width="0.3048" layer="1"/>
 </signal>
 <signal name="OE">
@@
 <signal name="G1">
 <contactref element="JP2" pad="6"/>
-<wire x1="18.415" y1="31.75" x2="17.78" y2="31.115" width="0.3048" layer="1"/>
+<wire x1="18.288" y1="31.75" x2="17.78" y2="31.115" width="0.3048" layer="1"/>
 <wire x1="17.78" y1="31.115" x2="16.51" y2="31.115" width="0.3048" layer="1"/>
 <contactref element="J1" pad="2"/>
-<via x="18.415" y="45.72" extent="1-16" drill="0.3556" diameter="0.7112"/>
-<wire x1="18.415" y1="45.72" x2="18.415" y2="46.355" width="0.3048" layer="16"/>
-<wire x1="18.415" y1="46.355" x2="20.955" y2="48.895" width="0.3048" layer="16"/>
-<wire x1="20.955" y1="48.895" x2="52.07" y2="48.895" width="0.3048" layer="16"/>
+<via x="18.288" y="45.847" extent="1-16" drill="0.3556" diameter="0.7112"/>
+<wire x1="18.288" y1="45.847" x2="21.336" y2="48.895" width="0.3048" layer="16"/>
+<wire x1="21.336" y1="48.895" x2="52.07" y2="48.895" width="0.3048" layer="16"/>
 <wire x1="52.07" y1="48.895" x2="52.705" y2="48.26" width="0.3048" layer="16"/>
 <wire x1="52.705" y1="48.26" x2="52.705" y2="47.371" width="0.3048" layer="16"/>
-<wire x1="18.415" y1="31.75" x2="18.415" y2="45.72" width="0" layer="19" extent="1-1"/>
+<wire x1="18.288" y1="31.75" x2="18.288" y2="37.592" width="0.3048" layer="1"/>
+<wire x1="18.288" y1="37.592" x2="17.145" y2="38.735" width="0.3048" layer="1"/>
+<wire x1="17.145" y1="38.735" x2="17.145" y2="44.704" width="0.3048" layer="1"/>
+<wire x1="17.145" y1="44.704" x2="18.288" y2="45.847" width="0.3048" layer="1"/>
 </signal>
 <signal name="E">

Commit message: Updated to V1.4
Parts:
- added JP1: JUMPER-SMT_2_NO_NO-SILK, SparkFun-Jumpers:SMT-JUMPER_2_NO_NO-SILK
- added R2: 4K7, _c2h:1/6W-RES
- added U2: DS18B20, SparkFun-Sensors:TO-92-AMMO
- moved R1 3.25 mm to (50.8, 38.9), turned to 180 degrees
- moved CN1 3.17 mm to (40.6, 4.45)
- moved X1 3.17 mm to (32.4, 8.89)
- moved J2 2.16 mm to (10.2, 9.91)
- moved U$1 2.01 mm to (47.6, 11.4)
- moved U1 1.80 mm to (50.8, 35.6), turned to 180 degrees
- moved U$3 1.40 mm to (49.7, 10.9)
Connections:
- removed net E: JP2.8, JP4.5, JP8.5
- new net DQ: JP1.2, JP4.5, JP8.5, R2.1, U2.2
- new net N$1: JP1.1, JP2.8
- net 3V3: now also R2.2, U2.3
- net GND: now also U2.1
Routing:
- net DQ: track 0.00 -> 75.8 mm, vias 0 -> 1
- net 3V3: track 38.8 -> 85.8 mm
- net E: track 38.2 -> 0.00 mm, vias 1 -> 0
- net 5V: track 62.3 -> 67.6 mm
- net A0: track 35.5 -> 37.3 mm
- net N$1: track 0.00 -> 1.50 mm
- net GND: vias 22 -> 23
Other:
- board size 45.1 x 47 mm -> 45.1 x 48.9 mm
- board text added: "R0 -- D7/GPIO13 E -/- D3/GPIO0 A --- D1/GPIO5 B --- D2/GPIO4 C --- D8/GPIO15 D --- D6/GPIO12 CLK - D5/GPIO14 STB - D0/GPIO16 OE -- D4/GPIO2"
- board text added: "WeMos Matrix Shield V1.4"
- board text removed: "R0 -- D7/GPIO13 E --- D7/GPIO0 A --- D1/GPIO5 B --- D2/GPIO4 C --- D8/GPIO15 D --- D6/GPIO12 CLK - D5/GPIO14 STB - D0/GPIO16 OE -- D4/GPIO2"
- board text removed: "WeMos Matrix Shield V1.3"

Commit message: Updated to V1.5
Parts:
- removed J3: (no value), SparkFun-Connectors:SCREWTERMINAL-3.5MM-4
- added X2: (no value), con-molex:KK-156-4
- moved U1 37.7 mm to (14.5, 45.7)
- moved R1 37.0 mm to (15.5, 49.9), turned to 0 degrees
- moved U$3 19.0 mm to (34.4, 22.4)
- moved U$1 18.2 mm to (31.1, 19.1)
- moved U2 14.0 mm to (40.6, 15.2)
- moved R2 6.94 mm to (44.6, 10.2), turned to 90 degrees
- moved J1 1.42 mm to (49.5, 48.6)
Connections:
- net 5V: now also X2.1, X2.2; no longer J3.1, J3.2
- net GND: now also X2.3, X2.4; no longer J3.3, J3.4
Routing:
- net A0: track 37.3 -> 15.1 mm
- net 3V3: track 85.8 -> 67.3 mm, vias 1 -> 2
- net G1: track 54.0 -> 48.1 mm
- net GND: track 2.54 -> 6.42 mm
- net 5V: track 67.6 -> 70.8 mm
- net DQ: track 75.8 -> 73.3 mm
- net B0: track 60.7 -> 58.3 mm
- net B1: track 53.9 -> 52.6 mm
- net R1: track 57.1 -> 58.3 mm
- net G0: track 42.8 -> 41.6 mm
Other:
- outline, holes or cut-outs redrawn
- board text added: "DQ"
- board text added: "V1.5"
- board text added: "WeMos Matrix Shield"
- board text added: "WeMos Matrix Shield V1.5"
- board text removed: "WeMos Matrix Shield V1.4"

Commit message: Updated to V1.6
Parts:
- added VIN1, VIN2, VIN3, VIN4: PADNORMAL, _c2h:PAD
- moved U2 31.1 mm to (9.53, 15.7)
- moved R2 26.8 mm to (18.4, 15.7), turned to 0 degrees
- moved U1 5.85 mm to (10.0, 49.5)
- moved C1 5.68 mm to (14.0, 44.5)
- moved JP2 5.68 mm to (8.89, 38.7)
- moved J2 5.43 mm to (5.08, 8.00)
- moved JP1 4.07 mm to (15.2, 31.1)
- moved JP4 3.59 mm to (41.9, 47.0)
- moved X1 3.59 mm to (29.8, 6.35)
- moved JP3 3.59 mm to (19.1, 47.0)
- moved JP7 3.59 mm to (21.6, 47.0)
- moved JP8 3.59 mm to (39.4, 47.0)
- moved U$3 3.18 mm to (31.9, 24.3)
- moved CN1 2.84 mm to (39.4, 1.91)
- moved J1 2.54 mm to (49.5, 51.2)
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Connections:
- new net SD3: VIN4.1
- new net SDO: VIN2.1
- new net TCK: VIN3.1
- new net TDO: VIN1.1
Routing:
- net 3V3: track 67.3 -> 77.9 mm
- net B: track 40.8 -> 51.2 mm
- net A: track 46.2 -> 56.6 mm
- net DQ: track 73.3 -> 65.9 mm, vias 1 -> 2
- net D: track 29.3 -> 36.6 mm
- net C: track 26.0 -> 33.3 mm
- net B0: track 58.3 -> 64.0 mm
- net R1: track 58.3 -> 63.9 mm
- net STB: track 37.5 -> 42.8 mm
- net G0: track 41.6 -> 46.7 mm
- net B1: track 52.6 -> 57.7 mm
- net G1: track 48.1 -> 53.1 mm
- net OE: track 38.5 -> 43.3 mm
- net R0: track 13.1 -> 15.7 mm
- net CLK: track 28.0 -> 30.6 mm
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Other:
- board size 45.1 x 48.9 mm -> 50.2 x 54 mm
- board text added: "V1.6"
- board text added: "WeMos Matrix Shield V1.6"
- board text removed: "V1.5"
- board text removed: "WeMos Matrix Shield V1.5"
